File: Circuit/Wood Badge circuit.kicad_pcb (KiCad board)
At the start: 2 copper layers, 60 x 60 mm, 12 parts, among them J1 Conn_01x02_Pin, U1 LM555xN

Commit message: Finished circuit. Submitted this desgin to PCBWay
Routing:
- net Net-(D2-K): track 0.00 -> 7.72 mm
Changed lines of the file:
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@@
       (outputformat 1)
       (mirror false)
-      (drillshape 1)
+      (drillshape 0)
       (scaleselection 1)
-      (outputdirectory "")
+      (outputdirectory "./240323-1 Flasher PCB")
     )
   )
@@
   (segment (start 62.04 44) (end 62.04 38.29) (width 0.25) (layer "B.Cu") (net 5))
   (segment (start 62.04 38.29) (end 63.5 36.83) (width 0.25) (layer "B.Cu") (net 5))
+  (segment (start 26.67 36.83) (end 26.67 42.67) (width 0.25) (layer "F.Cu") (net 6))
+  (segment (start 26.67 42.67) (end 28 44) (width 0.25) (layer "F.Cu") (net 6))
   (segment (start 50.8 34.29) (end 50.8 48.63) (width 0.25) (layer "F.Cu") (net 7))
   (segment (start 50.8 48.63) (end 48.62 50.81) (width 0.25) (layer "F.Cu") (net 7))
