File: Circuit/Wood Badge circuit.kicad_sch (KiCad schematic)
At the start: 10 parts, among them J1 Conn_01x02_Pin, U1 LM555xN

Commit message: Finished circuit. Submitted this desgin to PCBWay
Other:
- title: (none) -> LED Flasher
Changed lines of the file:
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@@
 (kicad_sch (version 20230121) (generator eeschema)
   (paper "A4")
+  (title_block
+    (title "LED Flasher")
+    (date "2024-03-23")
+    (rev "240323-1")
+  )
   (junction (at 166.37 45.085) (diameter 0) (color 0 0 0 0)
   )
