File: Circuit/Wood Badge circuit.kicad_sch (KiCad schematic)
At the start: 10 parts, among them J1 Conn_01x02_Pin, U1 LM555xN

Commit message: Added C3 (below R1, R2 oops) Added values of components to reach a 2Hz frequency
Parts:
- added C3: 10uF, Capacitor_THT:CP_Radial_D5.0mm_P2.50mm, symbol Device:C_Small
- C1: value C_Small -> 0.1uF
- C2: value C_Small -> 0.01uF
- R1, R2: value R_US -> 24KR
- R3, R4: value R_US -> 470R
Connections:
- net GND: now also C3.2
- net trigger-threshold: now also C3.1
Changed lines of the file:
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@@
+	)
+	(junction
+		(at 123.19 71.12)
+		(diameter 0)
+		(color 0 0 0 0)
 	)
 	(junction
@@
 	(wire
 		(pts
-			(xy 101.6 58.42) (xy 94.615 58.42)
+			(xy 52.07 53.975) (xy 69.215 53.975)
 		)
 		(stroke
@@
 	(wire
 		(pts
-			(xy 52.07 53.975) (xy 69.215 53.975)
+			(xy 142.875 55.245) (xy 142.875 59.69)
 		)
 		(stroke
@@
 	(wire
 		(pts
-			(xy 142.875 55.245) (xy 142.875 59.69)
+			(xy 158.75 45.085) (xy 166.37 45.085)
 		)
 		(stroke
@@
 	(wire
 		(pts
-			(xy 158.75 45.085) (xy 166.37 45.085)
+			(xy 142.875 64.77) (xy 142.875 69.215)
 		)
 		(stroke
@@
 	(wire
 		(pts
-			(xy 142.875 64.77) (xy 142.875 69.215)
+			(xy 94.615 63.5) (xy 123.19 63.5)
 		)
 		(stroke
@@
 	(wire
 		(pts
-			(xy 94.615 63.5) (xy 123.19 63.5)
+			(xy 123.19 63.5) (xy 123.19 62.865)
 		)
 		(stroke
@@
 	(wire
 		(pts
-			(xy 123.19 63.5) (xy 123.19 62.865)
+			(xy 94.615 68.58) (xy 111.125 68.58)
 		)
 		(stroke
@@
 	(wire
 		(pts
-			(xy 94.615 68.58) (xy 111.125 68.58)
+			(xy 166.37 43.815) (xy 166.37 45.085)
 		)
 		(stroke
@@
 	(wire
 		(pts
-			(xy 166.37 43.815) (xy 166.37 45.085)
+			(xy 111.125 68.58) (xy 111.125 71.12)
 		)
 		(stroke
@@
 	(wire
 		(pts
-			(xy 111.125 68.58) (xy 111.125 71.12)
+			(xy 111.125 71.12) (xy 123.19 71.12)
 		)
 		(stroke
@@
 	(wire
 		(pts
-			(xy 111.125 71.12) (xy 123.19 71.12)
+			(xy 94.615 58.42) (xy 101.6 58.42)
 		)
 		(stroke
@@
 			)
 		)
-		(property "Value" "R_US"
+		(property "Value" "470R"
 			(at 168.021 58.3621 0)
 			(effects
@@
 			)
 		)
-		(property "Value" "R_US"
+		(property "Value" "24KR"
 			(at 124.841 60.2671 0)
 			(effects
@@
 			)
 		)
-		(property "Value" "C_Small"
+		(property "Value" "0.01uF"
 			(at 66.6813 60.2178 90)
 			(effects
@@
 			)
 		)
-		(property "Value" "C_Small"
+		(property "Value" "0.1uF"
 			(at 145.1991 63.4484 0)
 			(effects
@@
 	)
 	(symbol
+		(lib_id "Device:C_Small")
+		(at 123.19 73.66 0)
+		(unit 1)
+		(exclude_from_sim no)
+		(in_bom yes)
+		(on_board yes)
+		(dnp no)
+		(fields_autoplaced yes)
+		(property "Reference" "C3"
+			(at 125.5141 72.4541 0)
+			(effects
+				(font
+					(size 1.27 1.27)
+				)
+				(justify left)
+			)
+		)
+		(property "Value" "10uF"
+			(at 125.5141 74.8784 0)
+			(effects
+				(font
+					(size 1.27 1.27)
+				)
+				(justify left)
+			)
+		)
+		(property "Footprint" "Capacitor_THT:CP_Radial_D5.0mm_P2.50mm"
+			(at 123.19 73.66 0)
+			(effects
+				(font
+					(size 1.27 1.27)
+				)
+				(hide yes)
+			)
+		)
+		(property "Datasheet" "~"
+			(at 123.19 73.66 0)
+			(effects
+				(font
+					(size 1.27 1.27)
+				)
+				(hide yes)
+			)
+		)
+		(property "Description" "Unpolarized capacitor, small symbol"
+			(at 123.19 73.66 0)
+			(effects
+				(font
+					(size 1.27 1.27)
+				)
+				(hide yes)
+			)
+		)
+		(pin "1"
+		)
+		(pin "2"
+		)
+		(instances
+			(project "Wood Badge circuit"
+				(path "/f8989166-43c6-4359-b996-a5eef05ca9de"
+					(reference "C3")
+					(unit 1)
+				)
+			)
+		)
+	)
+	(symbol
 		(lib_id "Device:R_US")
 		(at 123.19 67.31 0)
@@
 			)
 		)
-		(property "Value" "R_US"
+		(property "Value" "24KR"
 			(at 124.841 68.5221 0)
 			(effects
@@
 	)
 	(symbol
+		(lib_name "GND_1")
+		(lib_id "power:GND")
+		(at 123.19 76.2 0)
+		(unit 1)
+		(exclude_from_sim no)
+		(in_bom yes)
+		(on_board yes)
+		(dnp no)
+		(fields_autoplaced yes)
+		(property "Reference" "#PWR012"
+			(at 123.19 82.55 0)
+			(effects
+				(font
+					(size 1.27 1.27)
+				)
+				(hide yes)
+			)
+		)
+		(property "Value" "GND"
+			(at 123.19 80.3331 0)
+			(effects
+				(font
+					(size 1.27 1.27)
+				)
+			)
+		)
+		(property "Footprint" ""
+			(at 123.19 76.2 0)
+			(effects
+				(font
+					(size 1.27 1.27)
+				)
+				(hide yes)
+			)
+		)
+		(property "Datasheet" ""
+			(at 123.19 76.2 0)
+			(effects
+				(font
+					(size 1.27 1.27)
+				)
+				(hide yes)
+			)
+		)
+		(property "Description" "Power symbol creates a global label with name \"GND\" , ground"
+			(at 123.19 76.2 0)
+			(effects
+				(font
+					(size 1.27 1.27)
+				)
+				(hide yes)
+			)
+		)
+		(pin "1"
+		)
+		(instances
+			(project "Wood Badge circuit"
+				(path "/f8989166-43c6-4359-b996-a5eef05ca9de"
+					(reference "#PWR012")
+					(unit 1)
+				)
+			)
+		)
+	)
+	(symbol
 		(lib_id "Device:R_US")
 		(at 166.37 32.385 0)
@@
 		(fields_autoplaced yes)
 		(property "Reference" "R3"
-			(at 168.021 31.1729 0)
+			(at 168.021 31.1728 0)
 			(effects
 				(font
@@
 			)
 		)
-		(property "Value" "R_US"
+		(property "Value" "470R"
 			(at 168.021 33.5971 0)
 			(effects
